Commit message: Fixed URDF joints not working

File: src/reaper_description/urdf/URDFassy.urdf (robot description, URDF)
Before this commit: robot URDFassy, 3 links, 2 joints
Joints:
- removed joint Bucket
- removed joint Linkage
- added joint joint_Bucket: type revolute, parent Linkage, child Bucket, origin xyz=-0.29504 -0.29876 0 rpy=0 0 0.5499, axis 0 0 1, limit lower=-1.57 upper=1.57 effort=100 velocity=5.0
- added joint joint_Linkage: type revolute, parent Chassis, child Linkage, origin xyz=-0.33975 0 0.23217 rpy=1.5708 0.26832 0, axis 0 0 1, limit lower=-2.6 upper=0.4 effort=100 velocity=5.0

Commit message: fixed bounds on joints. now starts in starting configuration.

File: src/reaper_description/urdf/URDFassy.urdf (robot description, URDF)
Before this commit: robot URDFassy, 3 links, 2 joints
Joints:
- joint joint_Bucket: limit lower=-1.57 upper=1.57 effort=100 velocity=5.0 -> lower=-2.40 upper=1.05 effort=100 velocity=5.0
- joint joint_Linkage: limit lower=-2.6 upper=0.4 effort=100 velocity=5.0 -> lower=-3.1 upper=0.55 effort=100 velocity=5.0
